File: VCA_mix/vca_mix/vca_mix.kicad_pcb (KiCad board)
At the start: 2 copper layers, 190 parts, among them J1 power, J10 Thonkiconn, J11 Thonkiconn, J12 Thonkiconn, J13 Thonkiconn, J14 Thonkiconn, J2 Thonkiconn, J3 Thonkiconn, J4 Thonkiconn, J5 Thonkiconn, J6 Thonkiconn, J7 Thonkiconn, J8 Thonkiconn, J9 Thonkiconn, Q1 MMBT3904, Q10 MMBT3906, Q11 MMBT3904, Q12 MMBT3906, Q2 MMBT3906, Q3 MMBT3906, Q4 MMBT3906, Q5 MMBT3904, Q6 MMBT3906, Q7 MMBT3906, Q8 MMBT3904, Q9 MMBT3906, SW1 SW_SPDT, SW2 SW_SPDT, SW3 SW_SPDT, SW4 SW_SPDT, U1 LM13700, U10 LM4040DBZ-3, U2 LM13700, U3 TL072, U4 TL072, U5 TL074, U6 TL074, U7 TL074, U8 TL074, U9 TL072

Commit message: Rev 0 for common platform
Parts:
- moved RV4 141.1 mm to (64.3, 114.0), turned to 0 degrees
- moved R16 140.7 mm to (86.4, 119.4), turned to 90 degrees
- moved R17 139.0 mm to (88.6, 119.4), turned to -90 degrees
- moved C26 135.8 mm to (86.4, 58.7), turned to 0 degrees
- moved RV1 134.3 mm to (64.3, 108.2), turned to 0 degrees
- moved RV3 132.8 mm to (64.3, 75.2), turned to 0 degrees
- moved RV2 128.6 mm to (64.3, 69.1), turned to 0 degrees
- moved U3 128.0 mm to (71.4, 94.0)
- moved J1 124.0 mm to (71.6, 56.9)
- moved C25 121.4 mm to (61.5, 57.0)
- moved R14 121.2 mm to (84.1, 119.4), turned to 90 degrees
- moved R97 109.8 mm to (114.6, 159.8)
- moved R88 108.3 mm to (117.1, 153.2), turned to 90 degrees
- moved R95 107.6 mm to (83.8, 159.8)
- moved R96 107.5 mm to (99.1, 159.8)
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Routing:
- net +12V: track 0.00 -> 450.5 mm, vias 0 -> 21
- net -12V: track 0.00 -> 357.6 mm, vias 0 -> 13
- net VCA_1_IN: track 0.00 -> 97.9 mm, vias 0 -> 4
- net +3V0: track 0.00 -> 92.8 mm
- net Net-(U9A--): track 0.00 -> 91.5 mm, vias 0 -> 2
- net Net-(C17-Pad1): track 0.00 -> 86.2 mm, vias 0 -> 2
- net VCA_1_OUT: track 0.00 -> 78.7 mm, vias 0 -> 2
- net VCA_2_IN: track 0.00 -> 76.9 mm, vias 0 -> 2
- net Net-(C18-Pad1): track 0.00 -> 71.6 mm, vias 0 -> 3
- net VCA_3_IN: track 0.00 -> 66.9 mm, vias 0 -> 6
- net VCA_2_OUT: track 0.00 -> 66.8 mm, vias 0 -> 2
- net VCA_4_OUT: track 0.00 -> 65.9 mm, vias 0 -> 4
- net Net-(U5A--): track 0.00 -> 60.6 mm, vias 0 -> 2
- net Net-(C20-Pad1): track 0.00 -> 59.9 mm, vias 0 -> 1
- net Net-(U7A--): track 0.00 -> 59.6 mm, vias 0 -> 4
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- added copper zone on B.Cu, net GND
- added copper zone on F.Cu, net GND
