File: seed_common_platform/daisy_euro/daisy_euro.kicad_sch (KiCad schematic)
At the start: 33 parts, among them J1 thonkiconn, J10 thonkiconn, J2 thonkiconn, J3 thonkiconn, J4 thonkiconn, J5 thonkiconn, J6 thonkiconn, J7 thonkiconn, J8 thonkiconn, J9 thonkiconn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

Commit message: knob functionality added to board support
Other:
- note added: "ECO: Flip POT polarity, redraw for organization, add courtyard and silkscreen for power, change switches to minitaure"
Changed lines of the file:
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@@
     (stroke (width 0) (type default))
+  )
+  (text "ECO: Flip POT polarity, redraw for organization, \nadd courtyard and silkscreen for power, change \nswitches to minitaure"
+    (at 209.55 46.99 0)
+    (effects (font (size 1.27 1.27)) (justify left bottom))
   )
   (text "DAC" (at 20.32 49.53 0)
