File: Hardware/attenuverter_mixer/Mixer.kicad_sch (KiCad schematic)
At the start: 13 parts, among them J7 thonkiconn, SW1 SW_ON_ON_SPDT_MINI, U2 TL074

Commit message: created fabrication output
Parts:
- C3, C4: LCSC (none) -> C105622
- R15, R23, R24, R3: LCSC (none) -> C14675
- R18: LCSC (none) -> C83144
- R21, R22: LCSC (none) -> C137760
- U2: LCSC (none) -> C96507
Changed lines of the file:
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@@
+      (effects (font (size 1.27 1.27)) hide)
+    )
+    (property "LCSC" "C96507" (at 180.34 107.95 0)
       (effects (font (size 1.27 1.27)) hide)
     )
@@
       (effects (font (size 1.27 1.27)) hide)
     )
+    (property "LCSC" "C96507" (at 106.68 105.41 0)
+      (effects (font (size 1.27 1.27)) hide)
+    )
     (pin "1")
     (pin "2")
@@
       (effects (font (size 1.27 1.27)) hide)
     )
+    (property "LCSC" "C105622" (at 180.34 85.09 0)
+      (effects (font (size 1.27 1.27)) hide)
+    )
     (pin "1")
     (pin "2")
@@
       (effects (font (size 1.27 1.27)) hide)
     )
+    (property "LCSC" "C14675" (at 83.82 102.87 0)
+      (effects (font (size 1.27 1.27)) hide)
+    )
     (pin "1")
     (pin "2")
@@
     )
     (property "MPN" "865250442003" (at 135.89 96.52 0)
+      (effects (font (size 1.27 1.27)) hide)
+    )
+    (property "LCSC" "" (at 135.89 96.52 0)
       (effects (font (size 1.27 1.27)) hide)
     )
@@
     )
     (property "MPN" "RC0603FR-0724KL" (at 104.14 87.63 0)
+      (effects (font (size 1.27 1.27)) hide)
+    )
+    (property "LCSC" " C137760" (at 104.14 87.63 0)
       (effects (font (size 1.27 1.27)) hide)
     )
@@
       (effects (font (size 1.27 1.27)) hide)
     )
+    (property "LCSC" "C83144" (at 204.47 107.95 0)
+      (effects (font (size 1.27 1.27)) hide)
+    )
     (pin "1")
     (pin "2")
@@
       (effects (font (size 1.27 1.27)) hide)
     )
+    (property "LCSC" "C14675" (at 83.82 85.09 0)
+      (effects (font (size 1.27 1.27)) hide)
+    )
     (pin "1")
     (pin "2")
@@
       (effects (font (size 1.27 1.27)) hide)
     )
+    (property "LCSC" "C105622" (at 104.14 76.2 0)
+      (effects (font (size 1.27 1.27)) hide)
+    )
     (pin "1")
     (pin "2")
@@
       (effects (font (size 1.27 1.27)) hide)
     )
+    (property "LCSC" "C14675" (at 180.34 96.52 0)
+      (effects (font (size 1.27 1.27)) hide)
+    )
     (pin "1")
     (pin "2")
@@
     )
     (property "MPN" "RC0603FR-07100KL" (at 83.82 93.98 0)
+      (effects (font (size 1.27 1.27)) hide)
+    )
+    (property "LCSC" "C14675" (at 83.82 93.98 0)
       (effects (font (size 1.27 1.27)) hide)
     )
@@
       (effects (font (size 1.27 1.27)) hide)
     )
+    (property "LCSC" " C137760" (at 161.29 105.41 0)
+      (effects (font (size 1.27 1.27)) hide)
+    )

Commit message: proto order
Parts:
- removed C7: 10uF, Capacitor_SMD:CP_Elec_5x5.3, symbol synthesis:CAP_10UF_NONPOL
- added C8: 2.2uF, Capacitor_THT:C_Rect_L7.2mm_W4.5mm_P5.00mm_FKS2_FKP2_MKS2_MKP2, symbol synth:CAP_2.2UF_FILM
- SW1: now not fitted
- renumbered C3 to C7, C4 to C9, J7 to J6, R24 to R18, R23 to R19, R3 to R20, R15 to R23, R18 to R24
Connections:
- net at C7.2, R21.2, SW1.1 (A)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: now also C8.1
- net at SW1.3 (C): now also C8.2
