File: Hardware/attenuverter_mixer/attenuverter_mixer.kicad_pcb (KiCad board)
At the start: 4 copper layers, 48.8 x 107.9 mm, 57 parts, among them J1 thonkiconn, J2 thonkiconn, J3 thonkiconn, J4 thonkiconn, J5 thonkiconn, J6 thonkiconn, J7 euro_power_10, SW1 SW_ON_ON_SPDT_MINI, U1 TL074, U2 TL074

Commit message: proto order
Parts:
- C8: value 10uF -> 2.2uF; footprint Capacitor_SMD:CP_Elec_5x5.3 -> Capacitor_THT:C_Rect_L7.2mm_W4.5mm_P5.00mm_FKS2_FKP2_MKS2_MKP2
- moved C8 3.06 mm to (154.5, 87.5)
Routing:
- net Net-(SW1-A): track 55.7 -> 55.2 mm
