File: Hardware/output_module/output module/output module.kicad_pcb (KiCad board)
At the start: 2 copper layers, 0 parts

Commit message: rev A0 output module
Parts:
- added C1: 47pF, Capacitor_SMD:C_0603_1608Metric, B.Cu at (76.5, 76.6)
- added C10: 1uF, Capacitor_SMD:C_0603_1608Metric, B.Cu at (97.0, 142.6)
- added C11: 100nF, Capacitor_SMD:C_0603_1608Metric, B.Cu at (98.9, 147.2)
- added C12: 1uF, Capacitor_SMD:C_0603_1608Metric, B.Cu at (88.9, 148.8)
- added C13: 47pF, Capacitor_SMD:C_0603_1608Metric, B.Cu at (90.0, 86.6)
- added C14: 47pF, Capacitor_SMD:C_0603_1608Metric, B.Cu at (104.8, 86.9)
- added C15: 100nF, Capacitor_SMD:C_0603_1608Metric, B.Cu at (101.2, 102.2)
- added C16: 100nF, Capacitor_SMD:C_0603_1608Metric, B.Cu at (92.2, 102.2)
- added C17: 100nF, Capacitor_SMD:C_0603_1608Metric, B.Cu at (80.8, 77.7)
- added C18: 100nF, Capacitor_SMD:C_0603_1608Metric, B.Cu at (84.7, 77.7)
- added C19: 100nF, Capacitor_SMD:C_0603_1608Metric, B.Cu at (91.7, 83.7)
- added C2: 47pF, Capacitor_SMD:C_0603_1608Metric, B.Cu at (89.9, 72.0)
- added C20: 100nF, Capacitor_SMD:C_0603_1608Metric, B.Cu at (101.7, 83.4)
- added C21: 10uF, Capacitor_SMD:CP_Elec_5x5.3, B.Cu at (109.5, 58.8)
- added C22: 10uF, Capacitor_SMD:CP_Elec_5x5.3, B.Cu at (84.1, 59.1)
- added C23: 10uF, Capacitor_SMD:CP_Elec_5x5.3, B.Cu at (111.8, 73.3)
- added C24: 100nF, Capacitor_SMD:C_0603_1608Metric, B.Cu at (116.5, 99.1)
- added C25: 100nF, Capacitor_SMD:C_0603_1608Metric, B.Cu at (105.9, 94.9)
- added C26: 100nF, Capacitor_SMD:C_0603_1608Metric, B.Cu at (86.5, 95.5)
- added C27: 100nF, Capacitor_SMD:C_0603_1608Metric, B.Cu at (77.2, 98.9)
- added C3: 47pF, Capacitor_SMD:C_0603_1608Metric, B.Cu at (76.5, 67.7)
- added C4: 1uF, Capacitor_THT:C_Rect_L7.2mm_W4.5mm_P5.00mm_FKS2_FKP2_MKS2_MKP2, B.Cu at (75.9, 147.7)
- added C5: 1uF, Capacitor_THT:C_Rect_L7.2mm_W4.5mm_P5.00mm_FKS2_FKP2_MKS2_MKP2, B.Cu at (76.3, 138.5)
- added C6: 1uF, Capacitor_THT:C_Rect_L7.2mm_W4.5mm_P5.00mm_FKS2_FKP2_MKS2_MKP2, B.Cu at (92.2, 131.4)
- added C7: 1uF, Capacitor_THT:C_Rect_L7.2mm_W4.5mm_P5.00mm_FKS2_FKP2_MKS2_MKP2, B.Cu at (92.2, 136.8)
- added C8: 1uF, Capacitor_SMD:C_0603_1608Metric, B.Cu at (89.4, 145.7)
- added C9: 1uF, Capacitor_SMD:C_0603_1608Metric, B.Cu at (91.2, 142.1)
- added D1: 1N4148, Diode_SMD:D_SOD-323, B.Cu at (101.2, 100.3)
- added D10: 1N4148, Diode_SMD:D_SOD-323, B.Cu at (81.8, 112.1)
- added D11: 1N4148, Diode_SMD:D_SOD-323, B.Cu at (86.4, 112.1)
- added D12: GREEN, LED_THT:LED_D3.0mm, F.Cu at (90.0, 124.7)
- added D13: YELLOW, LED_THT:LED_D3.0mm, F.Cu at (84.1, 124.7)
- added D14: RED, LED_THT:LED_D3.0mm, F.Cu at (78.1, 124.7)
- added D2: 1N4148, Diode_SMD:D_SOD-323, B.Cu at (109.5, 112.1)
- added D3: 1N4148, Diode_SMD:D_SOD-323, B.Cu at (111.8, 112.1)
- added D4: 1N4148, Diode_SMD:D_SOD-323, B.Cu at (107.2, 112.1)
- added D5: GREEN, LED_THT:LED_D3.0mm, F.Cu at (103.5, 124.7)
- added D6: YELLOW, LED_THT:LED_D3.0mm, F.Cu at (109.5, 124.7)
- added D7: RED, LED_THT:LED_D3.0mm, F.Cu at (115.4, 124.7)
- added D8: 1N4148, Diode_SMD:D_SOD-323, B.Cu at (92.2, 100.3)
- added D9: 1N4148, Diode_SMD:D_SOD-323, B.Cu at (84.1, 112.1)
- added J1: thonkiconn, synthesis:thonkiconn, F.Cu at (80.1, 155.2)
- added J2: thonkiconn, synthesis:thonkiconn, F.Cu at (96.8, 155.2)
- added J3: thonkiconn, synthesis:thonkiconn, F.Cu at (113.6, 155.2)
- added J4: Conn_01x03, Connector_PinHeader_2.54mm:PinHeader_1x03_P2.54mm_Vertical, B.Cu at (109.4, 148.0)
- added J6: euro_power_16, synthesis:eurorack_16, B.Cu at (96.5, 66.7)
- added R1: 100k, Resistor_SMD:R_0603_1608Metric, B.Cu at (76.5, 73.0)
- added R10: 10k, Resistor_SMD:R_0603_1608Metric, B.Cu at (115.8, 65.0)
- added R11: 10k, Resistor_SMD:R_0603_1608Metric, B.Cu at (108.5, 87.0)
- added R12: 10k, Resistor_SMD:R_0603_1608Metric, B.Cu at (112.0, 87.0)
- added R13: 10k, Resistor_SMD:R_0603_1608Metric, B.Cu at (104.8, 112.0)
- added R14: 10k, Resistor_SMD:R_0603_1608Metric, B.Cu at (115.8, 115.8)
- added R15: 100k, Resistor_SMD:R_0603_1608Metric, B.Cu at (95.9, 91.1)
- added R16: 100k, Resistor_SMD:R_0603_1608Metric, B.Cu at (94.2, 91.1)
- added R17: 100k, Resistor_SMD:R_0603_1608Metric, B.Cu at (92.6, 91.1)
- added R18: 100k, Resistor_SMD:R_0603_1608Metric, B.Cu at (97.7, 91.1)
- added R19: 100k, Resistor_SMD:R_0603_1608Metric, B.Cu at (101.0, 91.1)
- added R2: 100k, Resistor_SMD:R_0603_1608Metric, B.Cu at (89.9, 70.2)
- added R20: 100k, Resistor_SMD:R_0603_1608Metric, B.Cu at (99.3, 91.1)
- added R21: 100k, Resistor_SMD:R_0603_1608Metric, B.Cu at (90.0, 88.3)
- added R22: 100k, Resistor_SMD:R_0603_1608Metric, B.Cu at (103.1, 86.9)
- added R23: 100k, Resistor_SMD:R_0603_1608Metric, B.Cu at (101.2, 105.5)
- added R24: 100k, Resistor_SMD:R_0603_1608Metric, B.Cu at (116.5, 95.8)
- added R25: 100k, Resistor_SMD:R_0603_1608Metric, B.Cu at (116.5, 100.7)
- added R26: 100k, Resistor_SMD:R_0603_1608Metric, B.Cu at (101.2, 98.4)
- added R27: 22k, Resistor_SMD:R_0603_1608Metric, B.Cu at (101.2, 107.2)
- added R28: 27k, Resistor_SMD:R_0603_1608Metric, B.Cu at (116.5, 97.4)
- added R29: 1k, Resistor_SMD:R_0603_1608Metric, B.Cu at (116.5, 102.4)
- added R3: 100k, Resistor_SMD:R_0603_1608Metric, B.Cu at (76.5, 71.2)
- added R30: 100k, Resistor_SMD:R_0603_1608Metric, B.Cu at (101.2, 96.7)
- added R31: 1k 0.5W, Resistor_SMD:R_1210_3225Metric, B.Cu at (103.5, 119.3)
- added R32: 1k 0.5W, Resistor_SMD:R_1210_3225Metric, B.Cu at (109.5, 119.3)
- added R33: 1k 0.5W, Resistor_SMD:R_1210_3225Metric, B.Cu at (115.4, 119.3)
- added R34: 100k, Resistor_SMD:R_0603_1608Metric, B.Cu at (101.2, 103.9)
- added R35: 100k, Resistor_SMD:R_0603_1608Metric, B.Cu at (77.2, 102.2)
- added R36: 100k, Resistor_SMD:R_0603_1608Metric, B.Cu at (77.2, 97.3)
- added R37: 100k, Resistor_SMD:R_0603_1608Metric, B.Cu at (92.2, 105.5)
- added R38: 100k, Resistor_SMD:R_0603_1608Metric, B.Cu at (92.2, 98.4)
- added R39: 22k, Resistor_SMD:R_0603_1608Metric, B.Cu at (77.2, 100.6)
- added R4: 68k, Resistor_SMD:R_0603_1608Metric, B.Cu at (76.5, 74.8)
- added R40: 27k, Resistor_SMD:R_0603_1608Metric, B.Cu at (77.2, 95.6)
- added R41: 1k, Resistor_SMD:R_0603_1608Metric, B.Cu at (92.2, 107.2)
- added R42: 100k, Resistor_SMD:R_0603_1608Metric, B.Cu at (92.2, 96.9)
- added R43: 1k 0.5W, Resistor_SMD:R_1210_3225Metric, B.Cu at (90.0, 119.3)
- added R44: 1k 0.5W, Resistor_SMD:R_1210_3225Metric, B.Cu at (84.1, 119.3)
- added R45: 1k 0.5W, Resistor_SMD:R_1210_3225Metric, B.Cu at (78.0, 119.3)
- added R46: 100k, Resistor_SMD:R_0603_1608Metric, B.Cu at (92.2, 103.9)
- added R5: 68k, Resistor_SMD:R_0603_1608Metric, B.Cu at (89.9, 73.8)
- added R6: 68k, Resistor_SMD:R_0603_1608Metric, B.Cu at (76.5, 69.5)
- added R7: 10k, Resistor_SMD:R_0603_1608Metric, B.Cu at (84.2, 134.7)
- added R8: 10k, Resistor_SMD:R_0603_1608Metric, B.Cu at (84.2, 136.5)
- added R9: 10k, Resistor_SMD:R_0603_1608Metric, B.Cu at (103.1, 65.0)
- added RV1: A100k, Potentiometer_THT:Potentiometer_Alpha_RD901F-40-00D_Single_Vertical, F.Cu at (81.6, 65.0)
- added RV2: A100k, Potentiometer_THT:Potentiometer_Alpha_RD901F-40-00D_Single_Vertical, F.Cu at (81.6, 90.4)
- added RV3: A100k, Potentiometer_THT:Potentiometer_Alpha_RD901F-40-00D_Single_Vertical, F.Cu at (81.6, 115.8)
- added RV4: A10K, Potentiometer_THT:Potentiometer_Alpha_RD902F-40-00D_Dual_Vertical, F.Cu at (81.6, 141.2)
- added RV5: 10k, Potentiometer_THT:Potentiometer_Alpha_RD901F-40-00D_Single_Vertical, F.Cu at (107.0, 65.0)
- added RV6: 10k, Potentiometer_THT:Potentiometer_Alpha_RD901F-40-00D_Single_Vertical, F.Cu at (107.0, 90.4)
- added RV7: 10k, Potentiometer_THT:Potentiometer_Alpha_RD901F-40-00D_Single_Vertical, F.Cu at (107.0, 115.8)
- added U1: TL074, Package_SO:TSSOP-14_4.4x5mm_P0.65mm, B.Cu at (82.8, 71.9)
- added U2: MAX97220C, Package_DFN_QFN:TQFN-16-1EP_3x3mm_P0.5mm_EP1.23x1.23mm, B.Cu at (93.7, 146.2)
- added U3: TL074, Package_SO:TSSOP-14_4.4x5mm_P0.65mm, B.Cu at (84.1, 99.8)
- added U4: TL074, Package_SO:TSSOP-14_4.4x5mm_P0.65mm, B.Cu at (109.5, 99.8)
- added U5: TL074, Package_SO:TSSOP-14_4.4x5mm_P0.65mm, B.Cu at (96.6, 85.0)
Routing:
- net +12V: track 0.00 -> 158.2 mm, vias 0 -> 10
- net Net-(J1-PadT): track 0.00 -> 104.6 mm, vias 0 -> 1
- net -12V: track 0.00 -> 100.6 mm, vias 0 -> 2
- net Net-(J3-PadT): track 0.00 -> 86.9 mm, vias 0 -> 1
- net chan_1: track 0.00 -> 82.4 mm, vias 0 -> 2
- net right_mix: track 0.00 -> 78.2 mm, vias 0 -> 2
- net chan_3: track 0.00 -> 77.9 mm, vias 0 -> 2
- net Net-(J2-PadT): track 0.00 -> 75.5 mm, vias 0 -> 2
- net GND: track 0.00 -> 72.8 mm, vias 0 -> 34
- net left_mix: track 0.00 -> 68.8 mm, vias 0 -> 2
- net chan_2: track 0.00 -> 56.2 mm, vias 0 -> 2
- net Net-(R3-Pad1): track 0.00 -> 52.6 mm, vias 0 -> 2
- net chan_1_right: track 0.00 -> 45.3 mm, vias 0 -> 1
- net chan_3_left: track 0.00 -> 40.5 mm, vias 0 -> 2
- net chan_1_left: track 0.00 -> 39.1 mm, vias 0 -> 1
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- added copper zone on In1.Cu, net +5V
- added copper zone on In2.Cu, net GND
Other:
- board outline added: 48.8 x 108 mm
- copper layers 2 -> 4
- board text added: "OUTPUT MODULE ISS-A SVG SYNTHESIS"

Commit message: update output module production mistakes
Parts:
- C4, C5, C6, C7: value 1uF -> 2.2uF; footprint Capacitor_THT:C_Rect_L7.2mm_W4.5mm_P5.00mm_FKS2_FKP2_MKS2_MKP2 -> synthesis:C_Rect_L7.8mm_W7.8mm_P5.00mm
- moved R10 12.8 mm to (103.0, 65.0), turned to 0 degrees
- moved R9 12.7 mm to (115.8, 65.0), turned to 180 degrees
- moved R13 11.7 mm to (115.8, 115.8), turned to 180 degrees
- moved R14 11.4 mm to (104.6, 113.6), turned to -90 degrees
- moved C5 11.1 mm to (74.2, 149.4), turned to 0 degrees
- moved C6 7.54 mm to (98.5, 127.3), turned to 180 degrees
- moved C4 6.65 mm to (82.3, 149.4)
- moved C7 6.58 mm to (98.8, 135.9), turned to 180 degrees
- moved R11 3.58 mm to (112.0, 86.6)
- moved R12 3.32 mm to (108.7, 86.6)
- moved C10 2.24 mm to (98.5, 144.3), turned to 0 degrees
- moved C12 2.16 mm to (90.4, 150.4), turned to -90 degrees
- moved C8 0.25 mm to (89.7, 145.7)
Connections:
- RV2 pad 2: Net-(R2-Pad1) -> Net-(R3-Pad1)
- RV3 pad 2: Net-(R3-Pad1) -> Net-(R2-Pad1)
- RV5 pad 1: chan_1_left -> chan_1_right
- RV5 pad 3: chan_1_right -> chan_1_left
- RV6 pad 1: chan_2_left -> chan_2_right
- RV6 pad 3: chan_2_right -> chan_2_left
- RV7 pad 1: chan_3_left -> chan_3_right
- RV7 pad 3: chan_3_right -> chan_3_left
Routing:
- net Net-(R2-Pad1): track 26.9 -> 53.3 mm
- net Net-(R3-Pad1): track 52.6 -> 29.7 mm
- net chan_1: track 82.4 -> 66.2 mm
- net chan_3_left: track 40.5 -> 49.3 mm, vias 2 -> 3
- net Net-(U2-INL+): track 15.5 -> 8.24 mm
- net Net-(C4-Pad1): track 15.7 -> 8.86 mm
- net Net-(C6-Pad1): track 22.2 -> 28.6 mm, vias 1 -> 0
- net Net-(U2-INL-): track 25.1 -> 20.4 mm
- net chan_3_right: track 39.0 -> 34.7 mm
- net chan_2_right: track 14.2 -> 10.3 mm
- net Net-(U2-INR+): track 14.6 -> 18.4 mm
- net GND: track 72.8 -> 69.3 mm
- net chan_1_left: track 39.1 -> 42.5 mm, vias 1 -> 2
- net chan_1_right: track 45.3 -> 43.3 mm
- net chan_2_left: track 22.7 -> 24.0 mm, vias 1 -> 0
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Other:
- board text added: "Revision History A: Initial Proto Order B: Corrected C4-7 footprint, fixed backwards pan pot, corrected PAN 2 and PAN3 swap"
