File: Hardware/output_module/output module/panning_mixer.kicad_sch (KiCad schematic)
At the start: 20 parts, among them U2 TL074

Commit message: proto order
Parts:
- RV5, RV6, RV7: now not fitted
- renumbered C15 to C13, C15 to C14, R3 to R15, R3 to R16, R3 to R17, R3 to R18, R3 to R19, R3 to R20, R3 to R21, R3 to R22, U2 to U1, U2 to U5

Commit message: update output module production mistakes
Parts:
- RV5, RV6, RV7: now fitted
Connections:
- net chan_1_left: now also RV5.3; no longer RV5.1
- net chan_1_right: now also RV5.1; no longer RV5.3
- net chan_2_left: now also RV6.3; no longer RV6.1
- net chan_2_right: now also RV6.1; no longer RV6.3
- net chan_3_left: now also RV7.3; no longer RV7.1
- net chan_3_right: now also RV7.1; no longer RV7.3
Changed lines of the file:
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@@
 	)
 	(junction
-		(at 71.12 120.65)
+		(at 93.98 135.89)
 		(diameter 0)
 		(color 0 0 0 0)
 	)
 	(junction
-		(at 69.85 52.07)
+		(at 93.98 101.6)
 		(diameter 0)
 		(color 0 0 0 0)
 	)
 	(junction
-		(at 93.98 86.36)
+		(at 71.12 120.65)
 		(diameter 0)
 		(color 0 0 0 0)
 	)
 	(junction
-		(at 218.44 140.97)
+		(at 69.85 52.07)
 		(diameter 0)
 		(color 0 0 0 0)
 	)
 	(junction
-		(at 193.04 59.69)
+		(at 93.98 120.65)
 		(diameter 0)
 		(color 0 0 0 0)
 	)
 	(junction
-		(at 194.31 128.27)
+		(at 92.71 52.07)
 		(diameter 0)
 		(color 0 0 0 0)
 	)
 	(junction
-		(at 71.12 86.36)
+		(at 92.71 67.31)
 		(diameter 0)
 		(color 0 0 0 0)
 	)
 	(junction
-		(at 93.98 135.89)
+		(at 218.44 140.97)
 		(diameter 0)
 		(color 0 0 0 0)
 	)
 	(junction
-		(at 93.98 101.6)
+		(at 193.04 59.69)
 		(diameter 0)
 		(color 0 0 0 0)
 	)
 	(junction
-		(at 93.98 120.65)
+		(at 194.31 128.27)
 		(diameter 0)
 		(color 0 0 0 0)
 	)
 	(junction
-		(at 217.17 72.39)
+		(at 71.12 86.36)
 		(diameter 0)
 		(color 0 0 0 0)
 	)
 	(junction
-		(at 218.44 128.27)
+		(at 217.17 72.39)
 		(diameter 0)
 		(color 0 0 0 0)
 	)
 	(junction
-		(at 194.31 118.11)
+		(at 218.44 128.27)
 		(diameter 0)
 		(color 0 0 0 0)
 	)
 	(junction
-		(at 92.71 52.07)
+		(at 194.31 118.11)
 		(diameter 0)
 		(color 0 0 0 0)
@@
 	)
 	(junction
-		(at 92.71 67.31)
+		(at 93.98 86.36)
 		(diameter 0)
 		(color 0 0 0 0)
@@
 	(wire
 		(pts
-			(xy 92.71 52.07) (xy 92.71 55.88)
-		)
-		(stroke
-			(width 0)
-			(type default)
-		)
-	)
-	(wire
-		(pts
-			(xy 92.71 67.31) (xy 104.14 67.31)
-		)
-		(stroke
-			(width 0)
-			(type default)
-		)
-	)
-	(wire
-		(pts
 			(xy 113.03 176.53) (xy 113.03 171.45)
 		)
@@
 	(wire
 		(pts
-			(xy 92.71 67.31) (xy 92.71 63.5)
+			(xy 200.66 49.53) (xy 193.04 49.53)
 		)
 		(stroke
@@
 	(wire
 		(pts
-			(xy 200.66 49.53) (xy 193.04 49.53)
+			(xy 200.66 59.69) (xy 193.04 59.69)
 		)
 		(stroke
@@
 	(wire
 		(pts
-			(xy 200.66 59.69) (xy 193.04 59.69)
+			(xy 93.98 86.36) (xy 93.98 90.17)
 		)
 		(stroke
@@
 	(wire
 		(pts
-			(xy 93.98 101.6) (xy 93.98 97.79)
+			(xy 97.79 93.98) (xy 101.6 93.98)
 		)
 		(stroke
@@
 	(wire
 		(pts
-			(xy 97.79 93.98) (xy 101.6 93.98)
+			(xy 217.17 49.53) (xy 217.17 59.69)
 		)
 		(stroke
@@
 	(wire
 		(pts
-			(xy 217.17 49.53) (xy 217.17 59.69)
+			(xy 93.98 135.89) (xy 105.41 135.89)
 		)
 		(stroke
@@
 	(wire
 		(pts
-			(xy 93.98 86.36) (xy 105.41 86.36)
+			(xy 83.82 86.36) (xy 93.98 86.36)
 		)
 		(stroke
@@
 	(wire
 		(pts
-			(xy 93.98 135.89) (xy 93.98 132.08)
-		)
-		(stroke
-			(width 0)
-			(type default)
-		)
-	)
-	(wire
-		(pts
 			(xy 193.04 69.85) (xy 196.85 69.85)
 		)
@@
 	(wire
 		(pts
-			(xy 92.71 52.07) (xy 104.14 52.07)
-		)
-		(stroke
-			(width 0)
-			(type default)
-		)
-	)
-	(wire
-		(pts
 			(xy 189.23 118.11) (xy 194.31 118.11)
 		)
@@
 	(wire
 		(pts
-			(xy 83.82 86.36) (xy 93.98 86.36)
-		)
-		(stroke
-			(width 0)
-			(type default)
-		)
-	)
-	(wire
-		(pts
 			(xy 71.12 120.65) (xy 76.2 120.65)
 		)
@@
 	(wire
 		(pts
-			(xy 93.98 101.6) (xy 105.41 101.6)
-		)
-		(stroke
-			(width 0)
-			(type default)
-		)
-	)
-	(wire
-		(pts
 			(xy 172.72 49.53) (xy 180.34 49.53)
 		)
@@
 	(wire
 		(pts
-			(xy 93.98 135.89) (xy 105.41 135.89)
+			(xy 63.5 176.53) (xy 60.96 176.53)
 		)
 		(stroke
@@
 	(wire
 		(pts
-			(xy 63.5 176.53) (xy 60.96 176.53)
+			(xy 82.55 52.07) (xy 92.71 52.07)
 		)
 		(stroke
@@
 	(wire
 		(pts
-			(xy 82.55 52.07) (xy 92.71 52.07)
+			(xy 189.23 138.43) (xy 194.31 138.43)
 		)
 		(stroke
@@
 	(wire
 		(pts
-			(xy 189.23 138.43) (xy 194.31 138.43)
+			(xy 93.98 120.65) (xy 105.41 120.65)
 		)
 		(stroke
@@
 	(wire
 		(pts
-			(xy 93.98 86.36) (xy 93.98 90.17)
+			(xy 93.98 101.6) (xy 105.41 101.6)
 		)
 		(stroke
@@
 	(wire
 		(pts
+			(xy 93.98 120.65) (xy 93.98 124.46)
+		)
+		(stroke
+			(width 0)
+			(type default)
+		)
+	)
+	(wire
+		(pts
 			(xy 101.6 93.98) (xy 101.6 95.25)
 		)
@@
 	(wire
 		(pts
+			(xy 93.98 97.79) (xy 93.98 101.6)
+		)
+		(stroke
+			(width 0)
+			(type default)
+		)
+	)
+	(wire
+		(pts
 			(xy 60.96 176.53) (xy 60.96 171.45)
 		)
@@
 	(wire
 		(pts
-			(xy 93.98 120.65) (xy 105.41 120.65)
+			(xy 83.82 120.65) (xy 93.98 120.65)
 		)
 		(stroke
@@
 	(wire
 		(pts
+			(xy 92.71 63.5) (xy 92.71 67.31)
+		)
+		(stroke
+			(width 0)
+			(type default)
+		)
+	)
+	(wire
+		(pts
 			(xy 194.31 128.27) (xy 194.31 138.43)
 		)
@@
 	(wire
 		(pts
-			(xy 83.82 120.65) (xy 93.98 120.65)
+			(xy 92.71 52.07) (xy 104.14 52.07)
 		)
 		(stroke
@@
 	(wire
 		(pts
+			(xy 92.71 52.07) (xy 92.71 55.88)
+		)
+		(stroke
+			(width 0)
+			(type default)
+		)
+	)
+	(wire
+		(pts
 			(xy 87.63 181.61) (xy 88.9 181.61)
 		)
@@
 	(wire
 		(pts
+			(xy 92.71 67.31) (xy 104.14 67.31)
+		)
+		(stroke
+			(width 0)
+			(type default)
+		)
+	)
+	(wire
+		(pts
 			(xy 187.96 69.85) (xy 193.04 69.85)
 		)
@@
 	(wire
 		(pts
+			(xy 93.98 132.08) (xy 93.98 135.89)
+		)
+		(stroke
+			(width 0)
+			(type default)
+		)
+	)
+	(wire
+		(pts
 			(xy 194.31 138.43) (xy 198.12 138.43)
 		)
@@
 	(wire
 		(pts
-			(xy 71.12 86.36) (xy 76.2 86.36)
+			(xy 93.98 86.36) (xy 105.41 86.36)
 		)
 		(stroke
@@
 	(wire
 		(pts
-			(xy 213.36 140.97) (xy 218.44 140.97)
+			(xy 71.12 86.36) (xy 76.2 86.36)
 		)
 		(stroke
@@
 	(wire
 		(pts
-			(xy 194.31 118.11) (xy 194.31 128.27)
+			(xy 213.36 140.97) (xy 218.44 140.97)
 		)
 		(stroke
@@
 	(wire
 		(pts
-			(xy 218.44 128.27) (xy 218.44 140.97)
+			(xy 194.31 118.11) (xy 194.31 128.27)
 		)
 		(stroke
@@
 	(wire
 		(pts
-			(xy 114.3 181.61) (xy 115.57 181.61)
+			(xy 218.44 128.27) (xy 218.44 140.97)
 		)
 		(stroke
@@
 	(wire
 		(pts
-			(xy 93.98 120.65) (xy 93.98 124.46)
+			(xy 114.3 181.61) (xy 115.57 181.61)
 		)
 		(stroke
@@
 		(lib_id "synthesis:ALPHAPOT_10K")
 		(at 93.98 93.98 0)
+		(mirror x)
 		(unit 1)
 		(exclude_from_sim no)
 		(in_bom yes)
 		(on_board yes)
-		(dnp yes)
+		(dnp no)
 		(property "Reference" "RV6"
-			(at 99.06 90.17 0)
+			(at 99.06 97.79 0)
 			(effects
 				(font
@@
 		)
 		(property "Value" "10k"
-			(at 99.06 96.52 0)
+			(at 99.06 91.44 0)
 			(effects
 				(font
@@
 		(lib_id "synthesis:ALPHAPOT_10K")
 		(at 93.98 128.27 0)
+		(mirror x)
 		(unit 1)
 		(exclude_from_sim no)
 		(in_bom yes)
 		(on_board yes)
-		(dnp yes)
+		(dnp no)
 		(property "Reference" "RV7"
-			(at 99.06 124.46 0)
+			(at 99.06 132.08 0)
 			(effects
 				(font
@@
 		)
 		(property "Value" "10k"
-			(at 99.06 130.81 0)
+			(at 99.06 125.73 0)
 			(effects
 				(font
@@
 		(lib_id "synthesis:ALPHAPOT_10K")
 		(at 92.71 59.69 0)
+		(mirror x)
 		(unit 1)
 		(exclude_from_sim no)
 		(in_bom yes)
 		(on_board yes)
-		(dnp yes)
+		(dnp no)
 		(property "Reference" "RV5"
-			(at 97.79 55.88 0)
+			(at 97.79 63.5 0)
 			(effects
 				(font
@@
 		)
 		(property "Value" "10k"
-			(at 97.79 62.23 0)
+			(at 97.79 57.15 0)
 			(effects
 				(font
