File: Hardware/seed_common_platform/daisy_euro/cv.kicad_sch (KiCad schematic)
At the start: 52 parts, among them U2 CD4052BPWR, U3 MCP6004, U6 MCP6004, U9 TL074CPWR

Commit message: fix rev A errors
Parts:
- renumbered C1 to C10, C1 to C11, C1 to C12, C1 to C13, C1 to C14, C1 to C15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
