File: Hardware/seed_common_platform/daisy_euro/daisy_euro.kicad_sch (KiCad schematic)
At the start: 33 parts, among them J1 thonkiconn, J10 thonkiconn, J2 thonkiconn, J3 thonkiconn, J4 thonkiconn, J5 thonkiconn, J6 thonkiconn, J7 thonkiconn, J8 thonkiconn, J9 thonkiconn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

Commit message: added ECO comments
Other:
- note added: "ECO: Flip POT polarity, redraw for organization, add courtyard and silkscreen for power, change switches to minitaure, space smd parts away from TH for manufacturability, increase hole size of daisy socket, new nomenclature for software alignment, make new switch, reposition LED, toggles, and button for UI"
- note removed: "ECO: Flip POT polarity, redraw for organization, add courtyard and silkscreen for power, change switches to minitaure"
Changed lines of the file:
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@@
     (stroke (width 0) (type default))
   )
-  (text "ECO: Flip POT polarity, redraw for organization, \nadd courtyard and silkscreen for power, change \nswitches to minitaure"
-    (at 209.55 46.99 0)
+  (text "ECO: Flip POT polarity, redraw for organization, \nadd courtyard and silkscreen for power, change \nswitches to minitaure, space smd parts away from TH \nfor manufacturability, increase hole size of daisy socket,\nnew nomenclature for software alignment, make new switch,\nreposition LED, toggles, and button for UI"
+    (at 209.55 50.8 0)
     (effects (font (size 1.27 1.27)) (justify left bottom))
   )
