File: Hardware/seed_common_platform/daisy_euro/power.kicad_sch (KiCad schematic)
At the start: 32 parts, among them J11 euro_power_10, U1 daisy_seed, U10 DG412DQ-T1-E3, U3 MCP6004, U4 TL074CPWR, U5 TL074CPWR, U6 MCP6004, U7 LM4040DBZ-10, U8 DG412DQ-T1-E3, U9 TL074CPWR

Commit message: fix rev A errors
Parts:
- renumbered C1 to C17, C1 to C18, C1 to C19, C1 to C20, C1 to C21, C1 to C22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
