File: Hardware/200_Plattform/200_Plattform.kicad_pcb (KiCad board)
At the start: 4 copper layers, 69.1 x 109.5 mm, 69 parts, among them J1 THONKICONN_MONO, J10 THONKICONN STEREO, J11 THONKICONN_MONO, J12 THONKICONN_MONO, J17 EURO_POWER_10_RTANG, J2 THONKICONN_MONO, J3 THONKICONN_MONO, J4 THONKICONN_MONO, J5 THONKICONN_MONO, J6 THONKICONN_MONO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

Commit message: board design review complete
Parts:
- moved RV5 2.59 mm to (73.0, 81.4)
- moved R17 1.02 mm to (72.6, 93.0)
- moved D2 1.02 mm to (74.4, 93.0)
- moved RV4 0.51 mm to (73.0, 54.1)
- moved D1 0.51 mm to (47.0, 111.8)
- moved J9 0.27 mm to (70.5, 118.9)
- moved J10 0.25 mm to (56.8, 118.9)
- moved J12 0.25 mm to (111.6, 139.2)
- moved J5 0.25 mm to (56.8, 139.2)
- moved J6 0.25 mm to (70.5, 139.2)
- moved J7 0.25 mm to (84.2, 139.2)
- moved J8 0.25 mm to (97.9, 139.2)
- moved J1 0.25 mm to (56.8, 129.0)
- moved J11 0.25 mm to (111.6, 129.0)
- moved J2 0.25 mm to (70.5, 129.0)
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- renumbered RV3 to RV2, RV5 to RV3, RV7 to RV4, RV2 to RV5, RV4 to RV6, RV6 to RV7
Routing:
- net in_1: track 80.6 -> 78.2 mm
- net pot_5: track 19.2 -> 21.6 mm
- net GATE_IN: track 15.9 -> 14.3 mm
- net AUDIO_LEFT: track 62.9 -> 61.6 mm
- net in_5: track 113.9 -> 112.9 mm
- net LED_LEFT: track 21.8 -> 22.8 mm
- net TACTILE_SW: track 68.6 -> 69.6 mm
- net pot_6: track 40.5 -> 41.3 mm
- net in_7: track 77.3 -> 78.0 mm
- net in_8: track 69.9 -> 70.5 mm
- net POT_MUX_B: track 33.0 -> 33.6 mm
- net Net-(D1-K): track 15.1 -> 14.6 mm
Other:
- board text added: "200 Series Platform Rev: A1"
