File: Hardware/200_Plattform/controls.kicad_sch (KiCad schematic)
At the start: 13 parts, among them SW1 SW_TACTILE, SW2 SW_SPDT_ON_OFF_ON_SUBMINI, SW3 SW_SPDT_ON_OFF_ON_SUBMINI, U4 CD4052B

Commit message: board design review complete
Parts:
- renumbered RV3 to RV2, RV5 to RV3, RV7 to RV4, RV2 to RV5, RV4 to RV6, RV6 to RV7
Changed lines of the file:
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@@
 		(dnp no)
 		(fields_autoplaced yes)
-		(property "Reference" "RV2"
+		(property "Reference" "RV5"
 			(at 39.37 88.8999 0)
 			(effects
@@
 			(project "200_Plattform"
 				(path "/74acaca0-79fd-4b91-90c4-143fa6f82a9e/29f1b18a-6032-4a1d-ae64-8a60aa88f83e"
-					(reference "RV2")
+					(reference "RV5")
 					(unit 1)
 				)
@@
 		(dnp no)
 		(fields_autoplaced yes)
-		(property "Reference" "RV6"
+		(property "Reference" "RV7"
 			(at 115.57 88.8999 0)
 			(effects
@@
 			(project "200_Plattform"
 				(path "/74acaca0-79fd-4b91-90c4-143fa6f82a9e/29f1b18a-6032-4a1d-ae64-8a60aa88f83e"
-					(reference "RV6")
+					(reference "RV7")
 					(unit 1)
 				)
@@
 		(dnp no)
 		(fields_autoplaced yes)
-		(property "Reference" "RV3"
+		(property "Reference" "RV2"
 			(at 77.47 57.1499 0)
 			(effects
@@
 			(project "200_Plattform"
 				(path "/74acaca0-79fd-4b91-90c4-143fa6f82a9e/29f1b18a-6032-4a1d-ae64-8a60aa88f83e"
-					(reference "RV3")
+					(reference "RV2")
 					(unit 1)
 				)
@@
 		(dnp no)
 		(fields_autoplaced yes)
-		(property "Reference" "RV5"
+		(property "Reference" "RV3"
 			(at 115.57 57.1499 0)
 			(effects
@@
 			(project "200_Plattform"
 				(path "/74acaca0-79fd-4b91-90c4-143fa6f82a9e/29f1b18a-6032-4a1d-ae64-8a60aa88f83e"
-					(reference "RV5")
+					(reference "RV3")
 					(unit 1)
 				)
@@
 		(dnp no)
 		(fields_autoplaced yes)
-		(property "Reference" "RV7"
+		(property "Reference" "RV4"
 			(at 153.67 57.1499 0)
 			(effects
@@
 			(project "200_Plattform"
 				(path "/74acaca0-79fd-4b91-90c4-143fa6f82a9e/29f1b18a-6032-4a1d-ae64-8a60aa88f83e"
-					(reference "RV7")
+					(reference "RV4")
 					(unit 1)
 				)
@@
 		(dnp no)
 		(fields_autoplaced yes)
-		(property "Reference" "RV4"
+		(property "Reference" "RV6"
 			(at 77.47 88.8999 0)
 			(effects
@@
 			(project "200_Plattform"
 				(path "/74acaca0-79fd-4b91-90c4-143fa6f82a9e/29f1b18a-6032-4a1d-ae64-8a60aa88f83e"
-					(reference "RV4")
-					(unit 1)
-				)
+					(reference "RV6")
+					(unit 1)
+				)
