File: Hardware/Source Files/200 Series/200_Plattform/controls.kicad_sch (KiCad schematic)
At the start: 13 parts, among them SW1 SW_TACTILE, SW2 SW_SPDT_ON_OFF_ON_SUBMINI, SW3 SW_SPDT_ON_OFF_ON_SUBMINI, U4 CD4052B

Commit message: Final Design Review 200 Series
Other:
- note added: "LEFT"
- note added: "RIGHT"
- moved on the sheet: SW3
Changed lines of the file:
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@@
+		)
+	)
+	(text "LEFT"
+		(exclude_from_sim no)
+		(at 103.886 156.718 0)
+		(effects
+			(font
+				(size 1.905 1.905)
+			)
+		)
+	)
+	(text "RIGHT"
+		(exclude_from_sim no)
+		(at 104.14 181.864 0)
+		(effects
+			(font
+				(size 1.905 1.905)
+			)
 		)
 	)
@@
 	(wire
 		(pts
-			(xy 90.17 163.83) (xy 93.98 163.83)
+			(xy 90.17 173.99) (xy 93.98 173.99)
 		)
 		(stroke
@@
 	(wire
 		(pts
-			(xy 104.14 166.37) (xy 107.95 166.37)
+			(xy 104.14 176.53) (xy 107.95 176.53)
 		)
 		(stroke
@@
 	(wire
 		(pts
-			(xy 90.17 165.1) (xy 90.17 163.83)
+			(xy 90.17 175.26) (xy 90.17 173.99)
 		)
 		(stroke
@@
 	(wire
 		(pts
-			(xy 104.14 161.29) (xy 107.95 161.29)
+			(xy 104.14 171.45) (xy 107.95 171.45)
 		)
 		(stroke
@@
 	(global_label "TOGGLE2_3"
 		(shape input)
-		(at 107.95 166.37 0)
-		(fields_autoplaced yes)
-		(effects
-			(font
-				(size 1.27 1.27)
-			)
-			(justify left)
-		)
-		(property "Intersheetrefs" "${INTERSHEET_REFS}"
-			(at 121.337 166.37 0)
+		(at 107.95 176.53 0)
+		(fields_autoplaced yes)
+		(effects
+			(font
+				(size 1.27 1.27)
+			)
+			(justify left)
+		)
+		(property "Intersheetrefs" "${INTERSHEET_REFS}"
+			(at 121.337 176.53 0)
 			(effects
 				(font
@@
 	(global_label "TOGGLE2_1"
 		(shape input)
-		(at 107.95 161.29 0)
-		(fields_autoplaced yes)
-		(effects
-			(font
-				(size 1.27 1.27)
-			)
-			(justify left)
-		)
-		(property "Intersheetrefs" "${INTERSHEET_REFS}"
-			(at 121.337 161.29 0)
+		(at 107.95 171.45 0)
+		(fields_autoplaced yes)
+		(effects
+			(font
+				(size 1.27 1.27)
+			)
+			(justify left)
+		)
+		(property "Intersheetrefs" "${INTERSHEET_REFS}"
+			(at 121.337 171.45 0)
 			(effects
 				(font
@@
 	(symbol
 		(lib_id "0_synthesis_other:SW_SPDT_ON_OFF_ON_SUBMINI")
-		(at 99.06 163.83 0)
+		(at 99.06 173.99 0)
 		(unit 1)
 		(exclude_from_sim no)
@@
 		(fields_autoplaced yes)
 		(property "Reference" "SW3"
-			(at 99.06 157.48 0)
+			(at 99.06 167.64 0)
 			(effects
 				(font
@@
 		)
 		(property "Value" "SW_SPDT_ON_OFF_ON_SUBMINI"
-			(at 99.06 168.91 0)
+			(at 99.06 179.07 0)
 			(effects
 				(font
@@
 		)
 		(property "Footprint" "0_synthesis_tht:SW_TOGGLE_2MS3T1B3M2QES"
-			(at 99.06 163.83 0)
+			(at 99.06 173.99 0)
 			(effects
 				(font
@@
 		)
 		(property "Datasheet" "~"
-			(at 99.06 171.45 0)
+			(at 99.06 181.61 0)
 			(effects
 				(font
@@
 		)
 		(property "Description" "SUBMINIATURE TOGGLE SWITCH ON OFF ON PC PIN"
-			(at 99.06 163.83 0)
+			(at 99.06 173.99 0)
 			(effects
 				(font
@@
 		)
 		(property "MFR" "DAILYWELL"
-			(at 99.06 163.83 0)
+			(at 99.06 173.99 0)
 			(effects
 				(font
@@
 		)
 		(property "MPN" "2MS3T1B1M2QES"
-			(at 99.06 163.83 0)
+			(at 99.06 173.99 0)
 			(effects
 				(font
@@
 		)
 		(property "LCSC" ""
-			(at 99.06 163.83 0)
+			(at 99.06 173.99 0)
 			(effects
 				(font
@@
 	(symbol
 		(lib_id "power:GND")
-		(at 90.17 165.1 0)
+		(at 90.17 175.26 0)
 		(unit 1)
 		(exclude_from_sim no)
@@
 		(fields_autoplaced yes)
 		(property "Reference" "#PWR065"
-			(at 90.17 171.45 0)
+			(at 90.17 181.61 0)
 			(effects
 				(font
@@
 		)
 		(property "Value" "GND"
-			(at 90.17 170.18 0)
+			(at 90.17 180.34 0)
 			(effects
 				(font
@@
 		)
 		(property "Footprint" ""
-			(at 90.17 165.1 0)
+			(at 90.17 175.26 0)
 			(effects
 				(font
@@
 		)
 		(property "Datasheet" ""
-			(at 90.17 165.1 0)
+			(at 90.17 175.26 0)
 			(effects
 				(font
@@
 		)
 		(property "Description" "Power symbol creates a global label with name \"GND\" , ground"
-			(at 90.17 165.1 0)
-			(effects
-				(font
+			(at 90.17 175.26 0)
+			(effects
+				(font
