File: Hardware/Source Files/200 Series/201_Blank_Faceplate/201_Blank_Faceplate.kicad_pcb (KiCad board)
At the start: 2 copper layers, 71.1 x 128.5 mm, 29 parts

Commit message: misc WIP
Other:
- board text added: "; DRILL file {KiCad 9.0.0} date 2025-04-07T22:14:04-0400 ; FORMAT={-:-/ absolute / inch / decimal} ; #@! TF.CreationDate,2025-04-07T22:14:04-04:00 ; #@! TF.GenerationSoftware,Kicad,Pcbnew,9.0.0 ; #@! TF.FileFunction,MixedPlating,1,2 FMAT,2 INCH ; #@! TA.AperFunction,NonPlated,NPTH,ComponentDrill T1C0.1150 ; #@! TA.AperFunction,NonPlated,NPTH,ComponentDrill T2C0.1260 ; #@! TA.AperFunction,NonPlate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"
