File: Hardware/Source Files/400 Series/401 VCO/AUDIO_IO.kicad_sch (KiCad schematic)
At the start: 33 parts, among them J11 THONKICONN_MONO, J2 THONKICONN_MONO, J3 THONKICONN_MONO, J4 THONKICONN_MONO, J5 THONKICONN_MONO, U3 TL074CPWR, U6 TL074CPWR, U9 TL074CPWR

Commit message: 404 VCA first pass layout/schematic
Parts:
- removed U3, U6: TL074CPWR, 0_synthesis_smt:TSSOP-14_4.4x5mm_P0.65mm, symbol 0_synthesis_ic:TL074CPWR
- added unit 4 of U1
- added unit 2 of U1
- added U3: TL074CPWR, 0_synthesis_smt:TSSOP-14_4.4x5mm_P0.65mm, symbol 0_synthesis_ic:TL074CPWR
- renumbered C21 to C15, C19 to C16, C20 to C17, C22 to C18, C34 to C19, J11 to J10, J4 to J6, J2 to J7, J3 to J8, J5 to J9, R31 to R45, R32 to R46, R24 to R47, R1 to R48, R27 to R49, R28 to R50, R33 to R51, R25 to R52, R29 to R53, R34 to R54, R26 to R55, R30 to R56, R35 to R57, R37 to R58, R58 to R59, R59 to R60, R36 to R61, R60 to R62, R38 to R63, R61 to R64, U9 to U1
Connections:
- net GND: now also U1.12 (+), U1.5 (+), U3.3 (+), U3.5 (+)
- net at C15.1, R45.2, R46.2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: now also U1.13 (-)
- net at C15.2, R51.2, R54.1: now also U1.14
- net at C16.1, R47.2, R48.2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: now also U3.6 (-)
- net at C17.1, R49.2, R50.2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: now also U3.2 (-)
- net at C17.2, R53.2, R56.1: now also U3.1
- net at C16.2, R52.2, R55.1: now also U3.7
- net at C18.2, R61.2, R63.1: now also U1.7
- net at C18.1, R57.2, R58.2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: now also U1.6 (-)
