File: Hardware/Source Files/400 Series/401 VCO/IO.kicad_sch (KiCad schematic)
At the start: 36 parts, among them J10 THONKICONN_MONO, J12 THONKICONN_MONO, J6 THONKICONN_MONO, J7 THONKICONN_MONO, J8 THONKICONN_MONO, J9 THONKICONN_MONO, SW2 SW_SPDT_ON_OFF_ON_SUBMINI, SW3 SW_Rotary_1x5_MP, SW4 SW_Rotary_1x5_MP, U10 TL074CPWR, U6 TL074CPWR, U9 TL074CPWR

Commit message: 404 VCA first pass layout/schematic
Parts:
- removed J9: THONKICONN_MONO, 0_synthesis_tht:JACK_THONKICONN_MONO_WQP518MA, symbol 0_synthesis_other:THONKICONN_MONO
- removed RV6, RV7, RV8: 10k, 0_synthesis_tht:ALPHAPOT, symbol 0_synthesis_other:POT_ALPHA_10K
- removed SW3, SW4: SW_Rotary_1x5_MP, symbol Switch:SW_Rotary_1x5_MP
- removed U10, U9: TL074CPWR, 0_synthesis_smt:TSSOP-14_4.4x5mm_P0.65mm, symbol 0_synthesis_ic:TL074CPWR
- added R40, R42, R43: 330R, 0_synthesis_smt:R_0603_1608Metric, symbol 0_synthesis_passives:RES_330R_0603
- added R44: 1k 0.5W, 0_synthesis_smt:R_1210_3225Metric, symbol 0_synthesis_passives:RES_1K_1210_0.5W
- added RV6, RV7, RV8: 10k, 0_synthesis_tht:Potentiometer_Slide_PTL30, symbol 0_synthesis_other:POT_SLIDE_30MM_RED_10K
- added SW3: SWITCH, 0_synthesis_tht:56DP36012AJN, symbol 0_synthesis_other:SW_Rotary_2x5_56DP36-01-2-AJN
- added U1: TL074CPWR, 0_synthesis_smt:TSSOP-14_4.4x5mm_P0.65mm, symbol 0_synthesis_ic:TL074CPWR
- added unit 3 of U5
- added U6: VREF_2.5V_0.2%, 0_synthesis_smt:SOT-23, symbol 0_synthesis_ic:VREF_2.5V_0.2%
- D1: renamed from D2; footprint Diode_SMD:D_SOD-323 -> 0_synthesis_smt:D_SOD-323
- D2: renamed from D1; footprint Diode_SMD:D_SOD-323 -> 0_synthesis_smt:D_SOD-323
- renumbered C32 to C10, C31 to C11, C33 to C12, C30 to C13, C35 to C14, J7 to J1, J6 to J2, J8 to J3, J12 to J4, J10 to J5, R41 to R29, R45 to R30, R46 to R31, R47 to R32, R48 to R33, R50 to R34, R44 to R35, R64 to R36, R54 to R37, R53 to R38, R51 to R39, R52 to R41, RV5 to RV4, RV3 to RV5, U6 to U5
Connections:
- net +5V: now also R40.1, R42.1, R43.1, RV8.1
- net -5VA: now also RV8.3
- net GND: now also RV6.3, RV6.E, RV7.3, RV7.E, RV8.E, SW3.5, U1.3 (+), U6.2 (A)
- net OCTAVE: now also U5.8, U5.9 (-)
- net PWM+: now also R44.2, U6.1 (K); no longer R41.2
- net TZFM_IN: now also RV6.2
- net PWM: now reaches J5.T, R39.1
- net at R37.2, R38.2, R39.2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: now also U1.2 (-)
- net AM_N1: now reaches C14.1
- net AM_N1: now also RV7.2
- net AM_N2: now reaches C14.2, R36.1
- net at R37.1: now also RV8.2
- net at R33.2, R34.1: now also SW3.4
- net at R30.2, R31.1: now also SW3.1
- net at R31.2, R32.1: now also SW3.2
- net at R32.2, R33.1: now also SW3.3
- net TZFM: now reaches J3.T
- net TZFM: now also RV6.1
- net SYNC: now reaches J1.T, SW2.2 (B)
- net AM: now reaches J4.T
- net AM: now also RV7.1
- new net: R40.2, RV8.B
- new net: R43.2, RV6.B
- new net: R41.2, R44.1, U1.1
- new net: R42.2, RV7.B
- new net: SW3.11, U5.10 (+)
Other:
- note removed: "AUXILIARY OUTPUT"
- moved on the sheet: R36
