File: Hardware/Source Files/400 Series/401 VCO/MODULATION.kicad_sch (KiCad schematic)
At the start: 20 parts, among them Q1 2N7002, SW1 SW_SPDT_ON_OFF_ON_SUBMINI, U3 TL074CPWR, U4 LM311

Commit message: 404 VCA first pass layout/schematic
Parts:
- removed U3: TL074CPWR, 0_synthesis_smt:TSSOP-14_4.4x5mm_P0.65mm, symbol 0_synthesis_ic:TL074CPWR
- added U3: TL074CPWR, 0_synthesis_smt:TSSOP-14_4.4x5mm_P0.65mm, symbol 0_synthesis_ic:TL074CPWR
- Q1: footprint Package_TO_SOT_SMD:SOT-23 -> 0_synthesis_smt:SOT-23
- U4: footprint Package_SO:SOIC-8_3.9x4.9mm_P1.27mm -> 0_synthesis_smt:SOIC-8_3.9x4.9mm_P1.27mm
- renumbered C15 to C5, C16 to C6, C13 to C7, C17 to C8, C14 to C9, R11 to R18, R12 to R19, R13 to R20, R17 to R21, R15 to R22, R14 to R23, R18 to R24, R19 to R25, R16 to R26, R20 to R27, R21 to R28
Connections:
- net GND: now also U3.12 (+)
- net at C7.1, R18.2, R19.2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: now also U3.13 (-)
- net at C7.2, R20.2, R22.1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: now also U3.14
- net at C9.2, R26.2, SW1.2 (B): now also U3.8
- net at Q1.3 (D), R23.2: now also U3.10 (+)
- net at C9.1, R22.2, R26.1: now also U3.9 (-)
