File: Hardware/Source Files/400 Series/401 VCO/SSI2130.kicad_sch (KiCad schematic)
At the start: 27 parts, among them U1 SSI2130, U11 TL074CPWR

Commit message: 404 VCA first pass layout/schematic
Parts:
- removed R5, R6: 22k, 0_synthesis_smt:R_0603_1608Metric, symbol 0_synthesis_passives:RES_22k_0603
- removed U11: TL074CPWR, 0_synthesis_smt:TSSOP-14_4.4x5mm_P0.65mm, symbol 0_synthesis_ic:TL074CPWR
- added C1: 100pF, 0_synthesis_smt:C_0603_1608Metric, symbol 0_synthesis_passives:CAP_100PF_0603_C0G
- added U5: TL074CPWR, 0_synthesis_smt:TSSOP-14_4.4x5mm_P0.65mm, symbol 0_synthesis_ic:TL074CPWR
- U2: renamed from U1; footprint Package_DFN_QFN:QFN-32-1EP_4x4mm_P0.4mm_EP2.65x2.65mm -> 0_synthesis_smt:QFN-32-1EP_4x4mm_P0.4mm_EP2.65x2.65mm
- renumbered C8 to C2, C9 to C3, C10 to C4, R55 to R1, R42 to R10, R43 to R11, R49 to R12, R39 to R13, R40 to R14, R9 to R15, R57 to R16, R7 to R17, R8 to R2, R56 to R3, R63 to R5, R62 to R6, R3 to R7, R2 to R8, R10 to R9, RV4 to RV2, RV2 to RV3
Connections:
- net GND: now also U5.12 (+)
- net BW_COMP: now reaches R17.1, U2.26 (BW_COMP)
- net SINE_IN-: now reaches R8.1, U2.3 (SINE_IN-)
- net at R1.2, R3.1: now also C1.1, U5.13 (-)
- net AUX_2_IN: now reaches R3.2, U2.5 (AUX_2_IN)
- net AUX_2_IN: now also C1.2, U5.14
- net AUX_2_MIX: now reaches R5.2, U2.13 (AUX_2_MIX)
- net SINE_IN+: now reaches R4.2, R7.1, U2.2 (SINE_IN+)
- net TCAP: now reaches C4.1, U2.14 (TCAP)
- net SQUARE: no longer names the net of U2.28 (SQUARE_OUT)
Other:
- moved on the sheet: R3, R4, R5, R6, R7, R8
