File: Hardware/Source Files/400 Series/403 VCF/403 VCF/403 VCF.kicad_sch (KiCad schematic)
At the start: 32 parts, among them J1 EURO_POWER_10_RTANG, J2 THONKICONN_MONO, J3 THONKICONN_MONO, U1 SSI2140

Commit message: fist pass 403VCF wip
Parts:
- removed C1, C3: 10uF, 0_synthesis_smt:C_P_2312_6032, symbol 0_synthesis_passives:CAP_10UF_TANTALUM
- removed C10, C7, C8, C9: 1nF, 0_synthesis_smt:C_0603_1608Metric, symbol 0_synthesis_passives:CAP_1NF_0603_C0G
- removed C2, C4, C5, C6: 100nF, 0_synthesis_smt:C_0603_1608Metric, symbol 0_synthesis_passives:CAP_100NF_0603_X7R
- removed D1, D2: MBR0530, 0_synthesis_smt:D_SOD-123, symbol 0_synthesis_ic:DIODE_MBR0530
- removed J1: EURO_POWER_10_RTANG, 0_synthesis_tht:EURO_POWER_10_RTANG, symbol 0_synthesis_other:EURO_POWER_10_RTANG
- removed J2, J3: THONKICONN_MONO, 0_synthesis_tht:JACK_THONKICONN_MONO_WQP518MA, symbol 0_synthesis_other:THONKICONN_MONO
- removed R1, R10, R11, R2, R4, R6, R7, R9: 10k, 0_synthesis_smt:R_0603_1608Metric, symbol 0_synthesis_passives:RES_10k_0603
- removed R12, R3, R5, R8: 220R, 0_synthesis_smt:R_0603_1608Metric, symbol 0_synthesis_passives:RES_220R_0603
- removed R13: 56k, 0_synthesis_smt:R_0603_1608Metric, symbol 0_synthesis_passives:RES_56k_0603
- removed R14: 15k, 0_synthesis_smt:R_0603_1608Metric, symbol 0_synthesis_passives:RES_15k_0603
- removed R15: 1k, 0_synthesis_smt:R_0603_1608Metric, symbol 0_synthesis_passives:RES_1K_0603
- removed R16: 1k 0.5W, 0_synthesis_smt:R_1210_3225Metric, symbol 0_synthesis_passives:RES_1K_1210_0.5W
- removed U1: SSI2140, 0_synthesis_smt:SSOP-20_4.4x6.5mm_P0.65mm, symbol 0_synthesis_ic:IC_SSI2140
Other:
- added sheet Filter (Filter.kicad_sch)
- added sheet IO (IO.kicad_sch)
- added sheet Power (Power.kicad_sch)
